File: board/pcb/lora-beetle-e1.kicad_pcb (KiCad board)
At the start: 2 copper layers, 56 x 101 mm, 10 parts, among them J1 BAT, J2 CubeCell J2, J3 CubeCell J3, J4 BME280 (GY-BME280), J5 BH1750 (GY-302)

Commit message: Project rename into Beetle E1
Other:
- board text added: "2026-10-17"
- board text added: "lora-beetle-e1"
- board text removed: "2026-10-16"
- board text removed: "lora-sensor-env1"
